Commit message: ...TODO: record the video..
TODO more:
if we wanna do a perfect job..
I suppose add workspace and divide the arm control and forward lateral control
is very necessary. since the planning is so unpredictable..

File: prius_description/urdf/prius.urdf (robot description, URDF)
Before this commit: robot prius, 24 links, 23 joints
Links:
- added link charge_oncar, mass 0.1; visual mesh filename=package://car_demo/models/charge_oncar/meshes/charge_oncar.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 scale=1 1 1
- added link charge_oncar::link_2, mass 0.01
Joints:
- added joint socket_connection_joint: type fixed, parent charge_oncar::link_2, child charge_oncar, origin xyz=0 0 0 rpy=0 0 0
- added joint socket_fake_joint: type fixed, parent base_link, child charge_oncar::link_2, origin xyz=-0.575 0.90 0.95 rpy=-1.35 0 0

Commit message: add realsense sensor to the end effector.. trying to use the vision based attaching method.

File: prius_description/urdf/prius.urdf (robot description, URDF)
Before this commit: robot prius, 26 links, 25 joints
Links:
- link charge_oncar: geometry visual mesh filename=package://prius_description/meshes/charge_oncar.dae scale=1 1 1
